Commit message: WIP: kuka_allegro_pose_fabric_example.py, allegro_pose_fabric_example.py: add finger tip attractors

File: src/fabrics_sim/models/robots/urdf/kuka_allegro/allegro.urdf (robot description, URDF)
Before this commit: robot allegro, 21 links, 20 joints
Links:
- added link index_link_1_sphere2
- added link index_link_3_sphere2
- added link middle_link_1_sphere2
- added link middle_link_3_sphere2
- added link palm_link_sphere2
- added link ring_link_1_sphere2
- added link ring_link_3_sphere2
- added link thumb_link_2_sphere2
- added link thumb_link_3_sphere2
- added link thumb_link_3_sphere3
Joints:
- added joint index_link_1_joint_sphere2: type fixed, parent index_link_1, child index_link_1_sphere2, origin xyz=0.027 0.0 0. rpy=0 0 0, axis 0 0 1
- added joint index_link_3_joint_sphere2: type fixed, parent index_link_3, child index_link_3_sphere2, origin xyz=0.035 0.005 0. rpy=0 0 0, axis 0 0 1
- added joint middle_link_1_joint_sphere2: type fixed, parent middle_link_1, child middle_link_1_sphere2, origin xyz=0.027 0.0 0. rpy=0 0 0, axis 0 0 1
- added joint middle_link_3_joint_sphere2: type fixed, parent middle_link_3, child middle_link_3_sphere2, origin xyz=0.035 0.005 0. rpy=0 0 0, axis 0 0 1
- added joint palm_link_joint_sphere2: type fixed, parent palm_link, child palm_link_sphere2, origin xyz=0 0.01 -0.05 rpy=0 0 0, axis 0 0 1
- added joint ring_link_1_joint_sphere2: type fixed, parent ring_link_1, child ring_link_1_sphere2, origin xyz=0.027 0.0 0. rpy=0 0 0, axis 0 0 1
- added joint ring_link_3_joint_sphere2: type fixed, parent ring_link_3, child ring_link_3_sphere2, origin xyz=0.035 0.005 0. rpy=0 0 0, axis 0 0 1
- added joint thumb_link_2_joint_sphere2: type fixed, parent thumb_link_2, child thumb_link_2_sphere2, origin xyz=0.025 0.0 0. rpy=0 0 0, axis 0 0 1
- added joint thumb_link_3_joint_sphere2: type fixed, parent thumb_link_3, child thumb_link_3_sphere2, origin xyz=0.025 0.0 0. rpy=0 0 0, axis 0 0 1
- added joint thumb_link_3_joint_sphere3: type fixed, parent thumb_link_3, child thumb_link_3_sphere3, origin xyz=0.055 0.005 0. rpy=0 0 0, axis 0 0 1
